Commit message: Fixed iK collisions

File: resources/2v2_2.1_1.2_1.1_8.10/hand/2v2_2.1_1.2_1.1_8.10.urdf (robot description, URDF)
Before this commit: robot 2v2_2.1_1.2_1.1_8.10, 7 links, 6 joints
Links:
- removed link finger0_sensor
- removed link finger1_sensor
Joints:
- removed joint finger0_sensor0_joint
- removed joint finger1_sensor1_joint
