Commit message: Ready for trials

File: resources/2v2_Demo/hand/2v2_Demo.urdf (robot description, URDF)
Before this commit: robot 2v2_Demo, 5 links, 4 joints
Joints:
- joint finger0_segment1_joint: origin xyz=0 0.072 0 rpy=0 0 0 -> xyz=0 0.07200000000000001 0 rpy=0 0 0
- joint finger1_segment1_joint: origin xyz=0 0.072 0 rpy=0 0 0 -> xyz=0 0.07200000000000001 0 rpy=0 0 0
